File: Node_Analog/Analog.kicad_sch (KiCad schematic)
At the start: 21 parts, among them J2 CONN_ANALOG, U11 TL431DBZ, U2 LM358

Commit message: New version.
Parts:
- removed J2: CONN_ANALOG, Connector_Phoenix_MC:PhoenixContact_MC_1,5_2-G-3.81_1x02_P3.81mm_Horizontal, symbol Connector_Generic:Conn_01x02
- added J2: CONN_ANALOG, Connector_Phoenix_MC:PhoenixContact_MC_1,5_4-G-3.81_1x04_P3.81mm_Horizontal, symbol Connector:Screw_Terminal_01x04
- added R22: 1K, Footprints:R_0603, symbol Device:R_Small
- added R23: 39K, Footprints:R_0603, symbol Device:R_Small
- R10: value 100R/1K -> 100R/220R
- R11: value 24K/10K -> 24K/8K2
- R35: value 100R/2K -> 1K/51R
- R36: value 8K2/DNP -> 82K
- R8: value 100R/DNP -> 100R/1uF
- R9: value 3K9/24K -> 1K/33K
- RV1, RV2: now not fitted
Connections:
- net GND: now also J2.2 (Pin_2), J2.3 (Pin_3)
- net at R36.2, RV2.3, U2.6 (-): now also R23.1
- net at C5.1, R8.2, R9.1: now also J2.4 (Pin_4)
- net at RV1.2, U2.1, U2.5 (+): now also R22.1
- net at R7.2, RV1.3, U2.2 (-): now also R22.2
- net at R37.1, RV2.2, U2.7: now also R23.2
- new net +24V: J2.1 (Pin_1)
Other:
- note added: "0-10V"
- note added: "2.5V"
- note added: "4-20mA"
- note added: "A1"
- note added: "A2"
- note added: "B1"
- note added: "B2"
- note added: "O"
- note added: "O1"
- note added: "O2"
- note added: "V"
- note removed: "0-10V:0R"
- note removed: "0-10V:1K"
- moved on the sheet: C33, C34, C35, C4, C5, D1, R10, R11, R35, R36, R37, R5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
