File: Node_Analog/ESP32-C3_BLE.kicad_sch (KiCad schematic)
At the start: 30 parts, among them J4 CONN_ESP_PROG, J5 USB_C_Receptacle_USB2.0_16P, Q2 SI2301, SW2 ESP-RESET, SW3 ESP-BOOT, U10 USBLC6-2SC6, U9 ESP32-C3, Y1 40MHz

Commit message: New version.
Parts:
- R25, R26, R27, R31: value 10K -> 20K
Changed lines of the file:
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@@
 			)
 		)
-		(property "Value" "10K"
+		(property "Value" "20K"
 			(at 196.088 76.2 0)
 			(effects
@@
 			)
 		)
-		(property "Value" "10K"
+		(property "Value" "20K"
 			(at 188.468 76.2 0)
 			(effects
@@
 			)
 		)
-		(property "Value" "10K"
+		(property "Value" "20K"
 			(at 59.182 69.85 0)
 			(effects
@@
 			)
 		)
-		(property "Value" "10K"
+		(property "Value" "20K"
 			(at 59.182 127 0)
 			(effects
