File: Node_Analog/Node_Analog.kicad_pcb (KiCad board)
At the start: 2 copper layers, 83.7 x 53.7 mm, 117 parts, among them J1 RAK_DEBUG, J2 CONN_ANALOG, J3 CONN_PWRIN, J4 CONN_ESP_PROG, J5 USB_C_Receptacle_USB2.0_16P, Q1 SI2300, Q2 SI2301, Q3 APM4015P, Q4 SI2300, Q5 SI2301, SW1 RAK-RESET, SW2 ESP-RESET, SW3 ESP-BOOT, SW4 USER_BTN, U1 RAK3172, U10 USBLC6-2SC6, U11 TL431DBZ, U12 DW01A, U13 FS8205A, U14 MT3608, U2 LM358, U3 BQ24075RGT, U4 XL1509-5.0, U5 TPS63000, U9 ESP32-C3, Y1 40MHz

Commit message: New version.
Parts:
- removed the   at (155.5, 70.6)
- removed C36: 100nF, Footprints:C_0603
- removed U12: DW01A, Footprints:SOT23-6
- removed U13: FS8205A, Package_SO:TSSOP-8_4.4x3mm_P0.65mm
- added  : LOGO, Footprints:LoGo_IoTVision_25x6.5, B.Cu at (130.6, 80.8)
- added C16: 1uF, Footprints:C_0603, F.Cu at (162.5, 86.6)
- added C17: 10uF, Footprints:C_0603, F.Cu at (174.5, 93.5)
- added C18: 10uF, Footprints:C_0603, F.Cu at (173.1, 93.5)
- added D6: SS34, Footprints:D_SMA, F.Cu at (170.8, 91.3)
- added L3: 22uH, Inductor_SMD:L_Bourns_SRN6045TA, F.Cu at (165.4, 91.3)
- added Q6: SI2300, Footprints:SOT23-3, F.Cu at (157.0, 91.4)
- added Q7: SI2301, Footprints:SOT23-3, F.Cu at (160.1, 87.0)
- added R22: 1K, Footprints:R_0603, F.Cu at (164.1, 75.2)
- added R23: 39K, Footprints:R_0603, F.Cu at (149.4, 75.3)
- added R24: 10R, Footprints:R_0603, F.Cu at (157.0, 87.4)
- added R32: 10K, Footprints:R_0603, F.Cu at (157.0, 88.8)
- added R33: 10K, Footprints:R_0603, F.Cu at (160.1, 89.6)
- added R34: 10R, Footprints:R_0603, F.Cu at (159.4, 91.7)
- added R38: 100K, Footprints:R_0603, F.Cu at (166.1, 83.8)
- added R39: 2K7, Footprints:R_0603, F.Cu at (163.2, 83.8)
- added R50: 0R, Footprints:R_0603, F.Cu at (148.7, 107.3)
- added U6: MT3608, Footprints:SOT23-6, F.Cu at (165.4, 86.0)
- J2: footprint Connector_Phoenix_MC:PhoenixContact_MC_1,5_2-G-3.81_1x02_P3.81mm_Horizontal -> Connector_Phoenix_MC:PhoenixContact_MC_1,5_4-G-3.81_1x04_P3.81mm_Horizontal
- R10: value 100R/1K -> 100R/220R
- R11: value 24K/10K -> 24K/8K2
- R19, R25, R26, R27, R3, R31: value 10K -> 20K
- R2: value 10K -> 100K
- R35: value 100R/2K -> 1K/51R
- R36: value 8K2/DNP -> 82K
- R43: value 100R -> 5K1
- R47: value 1K -> 0R
- R8: value 100R/DNP -> 100R/1uF
- R9: value 3K9/24K -> 1K/33K
- moved R43 39.8 mm to (169.0, 83.8)
- moved C37 26.8 mm to (138.6, 110.6), turned to 90 degrees
- moved R46 25.3 mm to (137.2, 110.6), turned to -90 degrees
- moved R45 23.9 mm to (135.8, 110.6), turned to 90 degrees
- moved R47 11.8 mm to (148.7, 105.9), turned to 180 degrees
- moved R40 6.50 mm to (138.3, 87.4), turned to 0 degrees
- moved RV1 5.72 mm to (164.1, 79.0)
- moved R37 5.67 mm to (145.9, 75.6)
- moved R7 5.66 mm to (159.9, 79.8)
- moved U2 5.66 mm to (156.2, 76.5)
- moved C34 5.66 mm to (153.8, 79.8)
- moved C35 5.66 mm to (142.0, 75.6)
- moved C4 5.66 mm to (159.2, 81.9)
- moved C5 5.66 mm to (160.7, 71.1)
- moved D1 5.66 mm to (143.9, 74.2)
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Connections:
- BT2 pad 2: -BATT -> GND
- C5 pad 1: Net-(J2-Pin_1) -> Net-(J2-Pin_4)
- J2 pad 1: Net-(J2-Pin_1) -> +24V
- R43 pad 1: +BATT -> +24V
- R47 pad 1: GND -> Net-(U5-PS/SYNC)
- R47 pad 2: Net-(U12-CS) -> GND
- R8 pad 2: Net-(J2-Pin_1) -> Net-(J2-Pin_4)
- R9 pad 1: Net-(J2-Pin_1) -> Net-(J2-Pin_4)
- U1 pad 10: unconnected-(U1-SDA/PA11-Pad10) -> /PSU/~{POWER_SAVE}
- U1 pad 13: unconnected-(U1-MOSI/PA7-Pad13) -> /PSU/5V_EN
- U1 pad 14: unconnected-(U1-MISO/PA6-Pad14) -> /PSU/24V_EN
- U1 pad 16: unconnected-(U1-SS/PA4-Pad16) -> /PSU/ACT_LED
- U1 pad 19: /PSU/ACT_LED -> unconnected-(U1-PA8-Pad19)
- U1 pad 27: /PSU/5V_EN -> unconnected-(U1-PB12-Pad27)
- U5 pad 7: Net-(U5-EN) -> Net-(U5-PS/SYNC)
Routing:
- net /PSU/~{POWER_SAVE}: track 0.00 -> 35.5 mm
- net /PSU/24V_EN: track 0.00 -> 29.2 mm, vias 0 -> 2
- net Net-(J2-Pin_1): track 28.0 -> 0.00 mm
- net Net-(J2-Pin_4): track 0.00 -> 27.5 mm
- net /PSU/VBAT_MONITOR: track 24.2 -> 50.8 mm
- net +BATT: track 35.8 -> 11.8 mm
- net /PSU/PPMIC_VOUT: track 79.3 -> 102.4 mm, vias 11 -> 13
- net +24V: track 0.00 -> 22.4 mm
- net /PSU/5V_EN: track 31.7 -> 10.9 mm
- net +3V3: track 136.9 -> 145.1 mm
- net -BATT: track 7.61 -> 0.00 mm
- net Net-(U5-PS/SYNC): track 0.00 -> 7.31 mm, vias 0 -> 2
- net /Analog/ANALOG_OUT: track 40.5 -> 35.5 mm
- net +5VA: track 21.8 -> 17.6 mm
- net Net-(D6-A): track 0.00 -> 4.14 mm
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- added copper zone on F.Cu, net Net-(D6-A)
- added copper zone on F.Cu, net Net-(Q7-D)
- removed copper zone on F.Cu, net +5VA
- removed copper zone on F.Cu, net -BATT
Other:
- board text added: "AIN GND GND VO"
- board text added: "B- B+"
- board text added: "CONFIG"
- board text added: "GND VCC"
- board text added: "LoRaWAN NODE ANALOG INTERFACE Mai Văn Anh - 20139059 Trần Đình Hoàng Anh - 20139061"
- board text removed: "+ -"
- board text removed: "GND AIN"
- board text removed: "LoRaWAN NODE ANALOG INTERFACE"
- board text removed: "USER"
