File: Node_Analog/Node_Analog.kicad_sch (KiCad schematic)
At the start: 0 parts

Commit message: New version.
Other:
- sheet PSU ports: added 24V_EN, ~{POWER_SAVE}; removed none
- sheet RAK3172_LoRa ports: added ANA_PWRON, ~{POWER_SAVE}; removed none
Changed lines of the file:
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@@
+	(wire
+		(pts
+			(xy 114.3 82.55) (xy 129.54 82.55)
+		)
+		(stroke
+			(width 0)
+			(type default)
+		)
+	)
 	(wire
 		(pts
@@
 			(width 0)
 			(type default)
+			(color 255 0 0 1)
+		)
+	)
+	(wire
+		(pts
+			(xy 114.3 78.74) (xy 129.54 78.74)
+		)
+		(stroke
+			(width 0)
+			(type default)
 		)
 	)
@@
 	(wire
 		(pts
-			(xy 114.3 77.47) (xy 129.54 77.47)
+			(xy 114.3 76.2) (xy 129.54 76.2)
 		)
 		(stroke
@@
 			(width 0)
 			(type default)
+		)
+	)
+	(netclass_flag ""
+		(length 2.54)
+		(shape round)
+		(at 173.99 96.52 0)
+		(fields_autoplaced yes)
+		(effects
+			(font
+				(size 1.27 1.27)
+			)
+			(justify left bottom)
+		)
+		(property "Netclass" "cc"
+			(at 174.6885 93.98 0)
+			(effects
+				(font
+					(size 1.27 1.27)
+					(italic yes)
+				)
+				(justify left)
+			)
 		)
 	)
@@
 		)
 		(pin "SENSOR_PWRON" output
-			(at 129.54 77.47 180)
+			(at 129.54 76.2 180)
 			(effects
 				(font
@@
 		(pin "ACT_LED" input
 			(at 129.54 86.36 180)
+			(effects
+				(font
+					(size 1.27 1.27)
+				)
+				(justify left)
+			)
+		)
+		(pin "ANA_PWRON" output
+			(at 129.54 78.74 180)
+			(effects
+				(font
+					(size 1.27 1.27)
+				)
+				(justify left)
+			)
+		)
+		(pin "~{POWER_SAVE}" output
+			(at 129.54 82.55 180)
 			(effects
 				(font
@@
 		)
 		(pin "5V_EN" input
-			(at 114.3 77.47 0)
+			(at 114.3 76.2 0)
 			(effects
 				(font
@@
 			(effects
 				(font
+					(size 1.27 1.27)
+				)
+				(justify right)
+			)
+		)
+		(pin "24V_EN" input
+			(at 114.3 78.74 0)
+			(effects
+				(font
+					(size 1.27 1.27)
+				)
+				(justify right)
+			)
+		)
+		(pin "~{POWER_SAVE}" input
+			(at 114.3 82.55 0)
+			(effects
+				(font
