File: Node_Analog/PSU.kicad_sch (KiCad schematic)
At the start: 51 parts, among them J3 CONN_PWRIN, Q3 APM4015P, Q4 SI2300, Q5 SI2301, U12 DW01A, U13 FS8205A, U14 MT3608, U3 BQ24075RGT, U4 XL1509-5.0, U5 TPS63000

Commit message: New version.
Parts:
- removed C36: 100nF, Footprints:C_0603, symbol Device:C_Small
- removed U12: DW01A, Footprints:SOT23-6, symbol Libraries:DW01A
- removed U13: FS8205A, Package_SO:TSSOP-8_4.4x3mm_P0.65mm, symbol Libraries:FS8205A
- added C16: 1uF, Footprints:C_0603, symbol Device:C_Small
- added C17, C18: 10uF, Footprints:C_0603, symbol Device:C_Small
- added D6: SS34, Footprints:D_SMA, symbol Diode:SS34
- added L3: 22uH, Inductor_SMD:L_Bourns_SRN6045TA, symbol Device:L_Ferrite
- added Q6: SI2300, Footprints:SOT23-3, symbol Transistor_FET:2N7002
- added Q7: SI2301, Footprints:SOT23-3, symbol Transistor_FET:AO3401A
- added R24, R34: 10R, Footprints:R_0603, symbol Device:R_Small
- added R32, R33: 10K, Footprints:R_0603, symbol Device:R_Small
- added R38: 100K, Footprints:R_0603, symbol Device:R_Small
- added R39: 2K7, Footprints:R_0603, symbol Device:R_Small
- added R50: 0R, Footprints:R_0603, symbol Device:R_Small
- added U6: MT3608, Footprints:SOT23-6, symbol Regulator_Switching:MT3608
- R43: value 100R -> 5K1
- R47: value 1K -> 0R; now not fitted
Connections:
- net -BATT is gone; now on net GND: BT2.2 (-)
- net +BATT: no longer R43.1
- net GND: now also R47.2, C16.1, C17.1, C18.1, Q6.2 (S), R32.2, R39.2, U6.2 (GND); no longer R47.1
- net PPMIC_VOUT: now also Q7.2 (S), R33.1
- net at C11.2, R16.2, U5.6 (EN)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: no longer U5.7 (PS/SYNC)
- net at R43.2: now also R38.1
- new net: Q6.1 (G), R24.2, R32.1
- new net: Q6.3 (D), R34.1
- new net: Q7.1 (G), R33.2, R34.2
- new net: R38.2, R39.1, U6.3 (FB)
- new net: R47.1, R50.1, U5.7 (PS/SYNC)
- new net: D6.2 (A), L3.2, U6.1 (SW)
- new net: C16.2, L3.1, Q7.3 (D), U6.4 (EN), U6.5 (IN)
- new net +24V: C17.2, C18.2, D6.1 (K), R43.1
- new net 24V_EN: R24.1
- new net ~{POWER_SAVE}: R50.2
- no-connect marks 3 -> 1
Other:
- note added: "3V3 buck-boost converter."
- note added: "7-40V to 5V buck converter."
- note added: "Boost converter for sensor."
- note removed: "8-40V TO 5V"
- note removed: "BOOST 5V (Analog)"
- note removed: "BUCK-BOOST TO 3V3"
- moved on the sheet: BT2, C11, C12, C37, C38, C39, C40, D2, L5, Q4, Q5, R16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
