File: Node_Analog/RAK3172_LoRa.kicad_sch (KiCad schematic)
At the start: 14 parts, among them J1 RAK_DEBUG, Q1 SI2300, SW1 RAK-RESET, SW4 USER_BTN, U1 RAK3172

Commit message: New version.
Parts:
- R19, R3: value 10K -> 20K
- R2: value 10K -> 100K
Connections:
- net ACT_LED: now also U1.16 (SS/PA4); no longer U1.19 (PA8)
- net SENSOR_PWRON: now also U1.13 (MOSI/PA7); no longer U1.27 (PB12)
- net ~{POWER_SAVE}: now reaches U1.10 (SDA/PA11)
- net ANA_PWRON: now reaches U1.14 (MISO/PA6)
- no-connect marks 14 -> 12
Changed lines of the file:
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@@
-	)
-	(no_connect
-		(at 198.12 90.17)
 	)
 	(no_connect
@@
 	)
 	(no_connect
-		(at 198.12 92.71)
+		(at 147.32 110.49)
 	)
 	(no_connect
@@
 	)
 	(no_connect
-		(at 198.12 77.47)
-	)
-	(no_connect
 		(at 198.12 105.41)
 	)
@@
 	)
 	(no_connect
-		(at 198.12 85.09)
+		(at 198.12 107.95)
 	)
 	(no_connect
@@
 	(hierarchical_label "SENSOR_PWRON"
 		(shape output)
-		(at 147.32 110.49 180)
+		(at 198.12 92.71 0)
 		(fields_autoplaced yes)
 		(effects
@@
 				(size 1.27 1.27)
 			)
-			(justify right)
+			(justify left)
 		)
 	)
@@
 		)
 	)
-	(hierarchical_label "ACT_LED"
-		(shape input)
-		(at 198.12 107.95 0)
+	(hierarchical_label "ANA_PWRON"
+		(shape output)
+		(at 198.12 90.17 0)
 		(fields_autoplaced yes)
 		(effects
@@
 		)
 	)
+	(hierarchical_label "ACT_LED"
+		(shape input)
+		(at 198.12 85.09 0)
+		(fields_autoplaced yes)
+		(effects
+			(font
+				(size 1.27 1.27)
+			)
+			(justify left)
+		)
+	)
 	(hierarchical_label "RAK_BOOT"
 		(shape input)
@@
 			)
 			(justify right)
+		)
+	)
+	(hierarchical_label "~{POWER_SAVE}"
+		(shape output)
+		(at 198.12 77.47 0)
+		(fields_autoplaced yes)
+		(effects
+			(font
+				(size 1.27 1.27)
+			)
+			(justify left)
 		)
 	)
@@
 			)
 		)
-		(property "Value" "10K"
+		(property "Value" "100K"
 			(at 90.932 83.82 0)
 			(effects
@@
 			)
 		)
-		(property "Value" "10K"
+		(property "Value" "20K"
 			(at 113.792 69.85 0)
 			(effects
 				(font
+					(face "KiCad Font")
 					(size 1.27 1.27)
 				)
@@
 			)
 		)
-		(property "Value" "10K"
+		(property "Value" "20K"
 			(at 220.218 107.95 0)
 			(effects
 				(font
-					(size 1.27 1.27)
-				)
+					(face "KiCad Font")
+					(size 1.27 1.27)
+				)
