File: Node_RS232/Node_RS232.kicad_pcb (KiCad board)
At the start: 2 copper layers, 83.7 x 53.7 mm, 103 parts, among them J1 RAK_DEBUG, J3 CONN_PWRIN, J4 CONN_ESP_PROG, J5 USB_C_Receptacle_USB2.0_16P, J6 CONN_RS232, Q1 SI2300, Q2 SI2301, Q3 SI2300, Q4 SI2301, Q5 APM4015P, SW1 RAK-RESET, SW2 ESP-RESET, SW3 ESP-BOOT, SW4 USER_BTN, U1 RAK3172, U10 USBLC6-2SC6, U2 MAX232, U3 BQ24075RGT, U4 XL1509-5.0, U5 TPS63000, U6 MT3608, U7 DW01A, U8 FS8205A, U9 ESP32-C3, Y1 40MHz

Commit message: New version.
Parts:
- removed the   at (154.7, 69.8)
- removed U7: DW01A, Footprints:SOT23-6
- removed U8: FS8205A, Package_SO:TSSOP-8_4.4x3mm_P0.65mm
- added  : LOGO, Footprints:LoGo_IoTVision_25x6.5, B.Cu at (163.5, 67.0)
- added Q6: SI2300, Footprints:SOT23-3, F.Cu at (161.0, 76.7)
- added Q7: SI2301, Footprints:SOT23-3, F.Cu at (168.8, 76.7)
- added R10: 0R, Footprints:R_0603, F.Cu at (149.3, 103.5)
- added R11: 10R, Footprints:R_0603, F.Cu at (157.0, 76.7)
- added R35: 10R, Footprints:R_0603, F.Cu at (163.5, 76.7)
- added R36: 4K7, Footprints:R_0603, F.Cu at (150.7, 81.4)
- added R9: 0R, Footprints:R_0603, F.Cu at (149.3, 104.9)
- C19: value 100nF -> 1uF
- R2, R33: value 10K -> 100K
- R21: value 20K -> 33K
- R23: value 100R -> 100K
- R24: value 1K -> 20K
- R25, R26, R27, R3, R31, R34, R7: value 10K -> 20K
- U2: value MAX232 -> MAX3232
- moved C19 41.9 mm to (164.9, 76.7), turned to -90 degrees
- moved R24 40.5 mm to (166.3, 76.7), turned to -90 degrees
- moved R23 34.2 mm to (158.4, 76.7), turned to -90 degrees
- moved C15 27.1 mm to (139.1, 108.4), turned to 90 degrees
- moved R20 25.6 mm to (137.7, 108.4), turned to -90 degrees
- moved R19 24.2 mm to (136.3, 108.4), turned to 90 degrees
- moved R32 6.82 mm to (138.8, 84.8), turned to 0 degrees
- moved R33 4.16 mm to (138.8, 86.2), turned to 180 degrees
- moved Q4 2.90 mm to (141.9, 84.5)
- moved R34 2.90 mm to (141.9, 87.1)
- moved R5 2.48 mm to (141.2, 89.2), turned to 90 degrees
- moved Q3 2.20 mm to (138.8, 88.8), turned to 90 degrees
- moved C11 0.70 mm to (150.0, 98.5)
Connections:
- BT1 pad 2: -BATT -> GND
- C17 pad 2: +5VD -> +9V
- C18 pad 2: +5VD -> +9V
- C19 pad 1: -BATT -> +3V3
- C19 pad 2: Net-(U7-VCC) -> GND
- C35 pad 2: +5VD -> Net-(Q7-D)
- D1 pad 1: +5VD -> +9V
- J6 pad 1: +5VD -> +9V
- R21 pad 1: +5VD -> Net-(R21-Pad1)
- R23 pad 1: +BATT -> Net-(Q6-G)
- R23 pad 2: Net-(U7-VCC) -> GND
- R24 pad 1: GND -> +3V3
- R32 pad 1: /PSU/5V_EN -> /PSU/9V_EN
- U1 pad 10: unconnected-(U1-SDA/PA11-Pad10) -> /PSU/~{POWER_SAVE}
- U1 pad 13: unconnected-(U1-MOSI/PA7-Pad13) -> /PSU/9V_EN
- U1 pad 16: unconnected-(U1-SS/PA4-Pad16) -> /PSU/LED_ACT
- U1 pad 19: /PSU/LED_ACT -> unconnected-(U1-PA8-Pad19)
- U1 pad 27: /PSU/5V_EN -> unconnected-(U1-PB12-Pad27)
- U1 pad 9: unconnected-(U1-SCL/PA12-Pad9) -> /RAK3172_LoRa/RS232_PWREN
- U2 pad 16: +5VD -> Net-(Q7-D)
- U5 pad 7: Net-(U5-EN) -> Net-(U5-PS/SYNC)
Routing:
- net +5VD: track 69.2 -> 0.00 mm
- net +9V: track 0.00 -> 42.0 mm
- net /PSU/~{POWER_SAVE}: track 0.00 -> 37.6 mm, vias 0 -> 2
- net /RAK3172_LoRa/RS232_PWREN: track 0.00 -> 33.3 mm
- net /PSU/5V_EN: track 32.2 -> 0.00 mm, vias 2 -> 0
- net /PSU/VBAT_MONITOR: track 24.6 -> 50.7 mm
- net +BATT: track 35.6 -> 11.2 mm
- net -BATT: track 15.0 -> 0.00 mm
- net Net-(Q7-D): track 0.00 -> 11.5 mm
- net /PSU/9V_EN: track 0.00 -> 10.4 mm, vias 0 -> 2
- net Net-(U5-PS/SYNC): track 0.00 -> 7.35 mm, vias 0 -> 2
- net Net-(Q7-G): track 3.29 -> 8.74 mm
- net /PSU/LED_ACT: track 48.3 -> 43.6 mm
- net Net-(Q4-D): track 14.6 -> 10.0 mm
- net Net-(U7-VCC): track 4.46 -> 0.00 mm
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- added copper zone on F.Cu, net +9V
- removed copper zone on F.Cu, net +5VD
- removed copper zone on F.Cu, net -BATT
Other:
- board text added: "B- B+"
- board text added: "CONFIG"
- board text added: "GND VCC"
- board text added: "LoRaWAN NODE RS232 INTERFACE Mai Văn Anh - 20139059 Trần Đình Hoàng Anh- 20139061"
- board text added: "TX RX GND VCC"
- board text removed: "+ -"
- board text removed: "LoRaWAN NODE RS232 INTERFACE"
- board text removed: "RX TX - +"
- board text removed: "USER"
