File: Node_RS232/Node_RS232.kicad_sch (KiCad schematic)
At the start: 0 parts

Commit message: New version.
Other:
- sheet PSU ports: added 9V_EN, ~{POWER_SAVE}; removed 5V_EN
- sheet RAK3172_LoRa ports: added RS232_PWREN, ~{POWER_SAVE}; removed none
- sheet RS232 ports: added RS232_EN; removed none
Changed lines of the file:
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@@
+	(wire
+		(pts
+			(xy 114.3 97.79) (xy 129.54 97.79)
+		)
+		(stroke
+			(width 0)
+			(type default)
+		)
+	)
 	(wire
 		(pts
@@
 	(wire
 		(pts
+			(xy 114.3 77.47) (xy 129.54 77.47)
+		)
+		(stroke
+			(width 0)
+			(type default)
+		)
+	)
+	(wire
+		(pts
 			(xy 114.3 72.39) (xy 129.54 72.39)
 		)
@@
 	(wire
 		(pts
-			(xy 114.3 77.47) (xy 129.54 77.47)
+			(xy 114.3 81.28) (xy 129.54 81.28)
 		)
 		(stroke
@@
 			)
 		)
+		(pin "~{POWER_SAVE}" output
+			(at 129.54 81.28 180)
+			(effects
+				(font
+					(size 1.27 1.27)
+				)
+				(justify left)
+			)
+		)
+		(pin "RS232_PWREN" output
+			(at 129.54 97.79 180)
+			(effects
+				(font
+					(size 1.27 1.27)
+				)
+				(justify left)
+			)
+		)
 		(instances
 			(project "Node_RS232"
@@
 			)
 		)
-		(pin "5V_EN" input
-			(at 114.3 77.47 0)
-			(effects
-				(font
-					(size 1.27 1.27)
-				)
-				(justify right)
-			)
-		)
 		(pin "LED_ACT" bidirectional
 			(at 114.3 86.36 0)
+			(effects
+				(font
+					(size 1.27 1.27)
+				)
+				(justify right)
+			)
+		)
+		(pin "9V_EN" input
+			(at 114.3 77.47 0)
+			(effects
+				(font
+					(size 1.27 1.27)
+				)
+				(justify right)
+			)
+		)
+		(pin "~{POWER_SAVE}" input
+			(at 114.3 81.28 0)
 			(effects
 				(font
@@
 			(effects
 				(font
+					(size 1.27 1.27)
+				)
+				(justify right)
+			)
+		)
+		(pin "RS232_EN" input
+			(at 114.3 97.79 0)
+			(effects
+				(font
