File: Node_RS232/PSU.kicad_sch (KiCad schematic)
At the start: 51 parts, among them J3 CONN_PWRIN, Q3 SI2300, Q4 SI2301, Q5 APM4015P, U3 BQ24075RGT, U4 XL1509-5.0, U5 TPS63000, U6 MT3608, U7 DW01A, U8 FS8205A

Commit message: New version.
Parts:
- removed C19: 100nF, Footprints:C_0603, symbol Device:C_Small
- removed R23: 100R, Footprints:R_0603, symbol Device:R_Small
- removed R24: 1K, Footprints:R_0603, symbol Device:R_Small
- removed U7: DW01A, Footprints:SOT23-6, symbol Libraries:DW01A
- removed U8: FS8205A, Package_SO:TSSOP-8_4.4x3mm_P0.65mm, symbol Libraries:FS8205A
- added R10, R9: 0R, Footprints:R_0603, symbol Device:R_Small
- added R36: 4K7, Footprints:R_0603, symbol Device:R_Small
- R21: value 20K -> 33K
- R33: value 10K -> 100K
- R34: value 10K -> 20K
Connections:
- net -BATT is gone; now on net GND: BT1.2 (-)
- net GND: now also R10.2
- net at C11.2, R16.2, U5.6 (EN)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: no longer U5.7 (PS/SYNC)
- net +5VD renamed +9V
- net +9V: now also R36.1; no longer R21.1
- net 5V_EN renamed 9V_EN
- new net: R21.1, R36.2
- new net: R10.1, R9.1, U5.7 (PS/SYNC)
- new net ~{POWER_SAVE}: R9.2
- no-connect marks 3 -> 1
Other:
- note added: "BOOST (RS232 & Sensor)"
- note removed: "BOOST 5V (RS232 Sensor)"
- moved on the sheet: C11, C12, C15, C16, C17, C18, D1, L3, Q3, Q4, R16, R19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
