File: Node_RS232/RS232.kicad_sch (KiCad schematic)
At the start: 7 parts, among them J6 CONN_RS232, U2 MAX232

Commit message: New version.
Parts:
- removed U2: MAX232, Footprints:SOIC-16-4x10-P1.27, symbol Interface_UART:MAX232
- added C19: 1uF, Footprints:C_0603, symbol Device:C_Small
- added Q6: SI2300, Footprints:SOT23-3, symbol Transistor_FET:2N7002
- added Q7: SI2301, Footprints:SOT23-3, symbol Transistor_FET:AO3401A
- added R11, R35: 10R, Footprints:R_0603, symbol Device:R_Small
- added R23: 100K, Footprints:R_0603, symbol Device:R_Small
- added R24: 20K, Footprints:R_0603, symbol Device:R_Small
- added U2: MAX3232, Footprints:SOIC-16-4x10-P1.27, symbol Interface_UART:MAX3232
Connections:
- net GND: now also C19.2, Q6.2 (S), R23.2, U2.15 (GND)
- net RS232_RX: now also U2.12 (R1OUT)
- net RS232_TX: now also U2.11 (T1IN)
- net at C33.1: now also U2.6 (VS-)
- net at J6.3 (Pin_3): now also U2.13 (R1IN)
- net at J6.4 (Pin_4): now also U2.14 (T1OUT)
- net at C34.1: now also U2.1 (C1+)
- net at C34.2: now also U2.3 (C1-)
- net at C5.1: now also U2.2 (VS+)
- net at C4.1: now also U2.4 (C2+)
- net at C4.2: now also U2.5 (C2-)
- net +5VD: no longer names the net of C35.2
- net +5VD: now also Q7.3 (D), U2.16 (VCC); no longer J6.1 (Pin_1)
- new net: Q6.1 (G), R11.2, R23.1
- new net: Q7.1 (G), R24.2, R35.2
- new net: Q6.3 (D), R35.1
- new net +3V3: C19.1, Q7.2 (S), R24.1
- new net +9V: J6.1 (Pin_1)
- new net RS232_EN: R11.1
