File: Node_RS485/Node_RS485.kicad_pcb (KiCad board)
At the start: 2 copper layers, 83.7 x 53.7 mm, 112 parts, among them J1 RAK_DEBUG, J2 CONN_RS485, J3 CONN_PWRIN, J4 CONN_ESP_PROG, J5 USB_C_Receptacle_USB2.0_16P, Q1 SI2300, Q2 SI2301, Q3 APM4015P, Q4 SI2300, Q5 SI2301, SW1 RAK-RESET, SW2 ESP-RESET, SW3 ESP-BOOT, SW4 USER_BTN, U1 RAK3172, U10 USBLC6-2SC6, U11 MT3608, U2 SP3485EN, U3 BQ24075RGT, U4 XL1509-5.0, U5 TPS63000, U7 DW01A, U8 FS8205A, U9 ESP32-C3, Y1 40MHz

Commit message: New version.
Parts:
- removed C19: 100nF, Footprints:C_0603
- removed U7: DW01A, Footprints:SOT23-6
- removed U8: FS8205A, Package_SO:TSSOP-8_4.4x3mm_P0.65mm
- added C17: 1uF, Footprints:C_0603, F.Cu at (165.6, 84.0)
- added Q6: SI2300, Footprints:SOT23-3, F.Cu at (161.7, 84.0)
- added Q7: SI2301, Footprints:SOT23-3, F.Cu at (169.5, 84.0)
- added R33: 0R, Footprints:R_0603, F.Cu at (158.2, 111.0)
- added R34: 10R, Footprints:R_0603, F.Cu at (157.7, 84.0)
- added R41: 100K, Footprints:R_0603, F.Cu at (159.1, 84.0)
- added R42: 20K, Footprints:R_0603, F.Cu at (167.0, 84.0)
- added R43: 10R, Footprints:R_0603, F.Cu at (164.2, 84.0)
- R2, R36: value 10K -> 100K
- R22, R25, R26, R27, R3, R31, R37: value 10K -> 20K
- R23: value 100R -> 4K7
- R24: value 1K -> 0R
- R39: value 51K -> 33K
- R8: value 4K7 -> 10R
- SW4: value USER_BTN -> MODE_SEL_BTN
- U2: value SP3485EN -> MAX3485EN
- moved C15 26.6 mm to (148.0, 115.8), turned to 90 degrees
- moved R23 25.7 mm to (159.7, 89.0)
- moved R20 25.2 mm to (146.6, 115.8), turned to -90 degrees
- moved R19 23.9 mm to (145.2, 115.8), turned to 90 degrees
- moved R24 11.8 mm to (158.2, 112.4), turned to 180 degrees
- moved R35 6.68 mm to (147.7, 92.4), turned to 0 degrees
- moved R36 4.01 mm to (147.7, 93.8), turned to 180 degrees
- moved R8 3.35 mm to (165.0, 87.2), turned to 0 degrees
- moved Q5 2.85 mm to (150.8, 92.1)
- moved R37 2.85 mm to (150.8, 94.7)
- moved R38 2.41 mm to (150.1, 96.8), turned to 90 degrees
- moved Q4 2.09 mm to (147.7, 96.3), turned to 90 degrees
- moved R6 1.90 mm to (165.0, 90.0)
- moved C11 0.70 mm to (158.9, 106.0)
- moved R5 0.20 mm to (165.0, 88.6)
Connections:
- BT1 pad 2: -BATT -> GND
- C34 pad 2: +12V -> +9V
- C35 pad 2: +12V -> +9V
- C4 pad 1: +3V3 -> Net-(Q7-D)
- C5 pad 1: +3V3 -> Net-(Q7-D)
- D7 pad 1: +12V -> +9V
- J2 pad 1: +12V -> +9V
- J5 pad A6: /ESP32-C3_BLE/ESP_USB_D_P -> /ESP32-C3_BLE/ESP_USB_D_N
- J5 pad A7: /ESP32-C3_BLE/ESP_USB_D_N -> Net-(U9-GPIO18/USB_D-)
- J5 pad B6: /ESP32-C3_BLE/ESP_USB_D_P -> /ESP32-C3_BLE/ESP_USB_D_N
- J5 pad B7: /ESP32-C3_BLE/ESP_USB_D_N -> Net-(U9-GPIO18/USB_D-)
- R23 pad 1: +BATT -> +9V
- R23 pad 2: Net-(U7-VCC) -> Net-(R23-Pad2)
- R24 pad 1: GND -> Net-(U5-PS/SYNC)
- R24 pad 2: Net-(U7-CS) -> /PSU/~{POWER_SAVE}
- R35 pad 1: /PSU/12V_EN -> /PSU/9V_EN
- R39 pad 1: +12V -> Net-(R23-Pad2)
- R5 pad 1: /RAK3172_LoRa/RS485_DR -> /RAK3172_LoRa/~{RS485_RE}
- R5 pad 2: Net-(U2-DE) -> Net-(U2-~{RE})
- R8 pad 1: Net-(U2-RO) -> /RAK3172_LoRa/RS485_DE
- R8 pad 2: +3V3 -> Net-(U2-DE)
- U1 pad 10: unconnected-(U1-SDA/PA11-Pad10) -> /PSU/~{POWER_SAVE}
- U1 pad 13: unconnected-(U1-MOSI/PA7-Pad13) -> /PSU/9V_EN
- U1 pad 14: unconnected-(U1-MISO/PA6-Pad14) -> /RAK3172_LoRa/~{RS485_RE}
- U1 pad 15: unconnected-(U1-SCK/PA5-Pad15) -> /RAK3172_LoRa/RS485_DE
- U1 pad 16: unconnected-(U1-SS/PA4-Pad16) -> /PSU/LED_ACT
- U1 pad 19: /PSU/LED_ACT -> unconnected-(U1-PA8-Pad19)
- U1 pad 27: /PSU/12V_EN -> unconnected-(U1-PB12-Pad27)
- U1 pad 6: /RAK3172_LoRa/RS485_DR -> unconnected-(U1-PA1-Pad6)
- U1 pad 9: unconnected-(U1-SCL/PA12-Pad9) -> /RAK3172_LoRa/RS485_PWREN
- U10 pad 1: /ESP32-C3_BLE/ESP_USB_D_N -> Net-(U9-GPIO18/USB_D-)
- U10 pad 3: /ESP32-C3_BLE/ESP_USB_D_P -> /ESP32-C3_BLE/ESP_USB_D_N
- U10 pad 4: /ESP32-C3_BLE/ESP_USB_D_P -> /ESP32-C3_BLE/ESP_USB_D_N
- U10 pad 6: /ESP32-C3_BLE/ESP_USB_D_N -> Net-(U9-GPIO18/USB_D-)
- U2 pad 2: Net-(U2-DE) -> Net-(U2-~{RE})
- U2 pad 8: +3V3 -> Net-(Q7-D)
- U5 pad 7: Net-(U5-EN) -> Net-(U5-PS/SYNC)
- U9 pad 25: /ESP32-C3_BLE/ESP_USB_D_N -> Net-(U9-GPIO18/USB_D-)
- U9 pad 26: /ESP32-C3_BLE/ESP_USB_D_P -> /ESP32-C3_BLE/ESP_USB_D_N
Routing:
- net +12V: track 43.6 -> 0.00 mm
- net +9V: track 0.00 -> 41.0 mm
- net /RAK3172_LoRa/RS485_DR: track 38.4 -> 0.00 mm
- net /PSU/~{POWER_SAVE}: track 0.00 -> 37.5 mm, vias 0 -> 2
- net /PSU/12V_EN: track 31.9 -> 0.00 mm, vias 2 -> 0
- net /PSU/VBAT_MONITOR: track 24.4 -> 52.1 mm
- net /RAK3172_LoRa/RS485_PWREN: track 0.00 -> 24.9 mm, vias 0 -> 2
- net +BATT: track 39.4 -> 14.5 mm
- net Net-(U9-GPIO18/USB_D-): track 0.00 -> 24.7 mm
- net /ESP32-C3_BLE/ESP_USB_D_P: track 23.7 -> 0.00 mm
- net /RAK3172_LoRa/~{RS485_RE}: track 0.00 -> 23.3 mm
- net /RAK3172_LoRa/RS485_DE: track 0.00 -> 23.1 mm
- net -BATT: track 15.2 -> 0.00 mm
- net /PSU/9V_EN: track 0.00 -> 10.7 mm, vias 0 -> 2
- net Net-(Q7-D): track 0.00 -> 9.34 mm
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- added copper zone on F.Cu, net +9V
- removed copper zone on F.Cu, net +12V
- removed copper zone on F.Cu, net -BATT
Other:
- board text added: "B- B+"
- board text added: "CONFIG"
- board text added: "LoRaWAN NODE RS485 INTERFACE Mai Văn Anh - 20139059 Trần Đình Hoàng Anh- 20139061"
- board text removed: "LoRaWAN NODE RS485 INTERFACE"
- board text removed: "USER"
