File: Node_RS485/Node_RS485.kicad_sch (KiCad schematic)
At the start: 0 parts

Commit message: New version.
Other:
- sheet PSU ports: added 9V_EN, ~{POWER_SAVE}; removed 12V_EN
- sheet RAK3172_LoRa ports: added RS485_DE, RS485_PWREN, ~{POWER_SAVE}, ~{RS485_RE}; removed RS485_DR
- sheet RS485 ports: added RS485_DE, RS485_EN, ~{RS485_RE}; removed RS485_DR
Changed lines of the file:
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@@
 	(wire
 		(pts
-			(xy 114.3 106.68) (xy 129.54 106.68)
+			(xy 114.3 109.22) (xy 129.54 109.22)
 		)
 		(stroke
@@
 	(wire
 		(pts
+			(xy 114.3 104.14) (xy 129.54 104.14)
+		)
+		(stroke
+			(width 0)
+			(type default)
+		)
+	)
+	(wire
+		(pts
+			(xy 114.3 97.79) (xy 129.54 97.79)
+		)
+		(stroke
+			(width 0)
+			(type default)
+		)
+	)
+	(wire
+		(pts
 			(xy 182.88 96.52) (xy 167.64 96.52)
 		)
@@
 	(wire
 		(pts
+			(xy 114.3 81.28) (xy 129.54 81.28)
+		)
+		(stroke
+			(width 0)
+			(type default)
+		)
+	)
+	(wire
+		(pts
 			(xy 182.88 106.68) (xy 167.64 106.68)
 		)
@@
 	(wire
 		(pts
-			(xy 114.3 109.22) (xy 129.54 109.22)
-		)
-		(stroke
-			(width 0)
-			(type default)
-		)
-	)
-	(wire
-		(pts
-			(xy 114.3 99.06) (xy 129.54 99.06)
+			(xy 114.3 111.76) (xy 129.54 111.76)
+		)
+		(stroke
+			(width 0)
+			(type default)
+		)
+	)
+	(wire
+		(pts
+			(xy 114.3 100.33) (xy 129.54 100.33)
 		)
 		(stroke
@@
 		)
 		(pin "RS485_RX" input
-			(at 129.54 106.68 180)
+			(at 129.54 109.22 180)
 			(effects
 				(font
@@
 		)
 		(pin "RS485_TX" output
-			(at 129.54 109.22 180)
-			(effects
-				(font
-					(size 1.27 1.27)
-				)
-				(justify left)
-			)
-		)
-		(pin "RS485_DR" output
-			(at 129.54 99.06 180)
+			(at 129.54 111.76 180)
 			(effects
 				(font
@@
 		(pin "LED_ACT" bidirectional
 			(at 129.54 86.36 180)
+			(effects
+				(font
+					(size 1.27 1.27)
+				)
+				(justify left)
+			)
+		)
+		(pin "~{RS485_RE}" output
+			(at 129.54 100.33 180)
+			(effects
+				(font
+					(size 1.27 1.27)
+				)
+				(justify left)
+			)
+		)
+		(pin "RS485_DE" output
+			(at 129.54 97.79 180)
+			(effects
+				(font
+					(size 1.27 1.27)
+				)
+				(justify left)
+			)
+		)
+		(pin "~{POWER_SAVE}" output
+			(at 129.54 81.28 180)
+			(effects
+				(font
+					(size 1.27 1.27)
+				)
+				(justify left)
+			)
+		)
+		(pin "RS485_PWREN" output
+			(at 129.54 104.14 180)
 			(effects
 				(font
@@
 			)
 		)
-		(pin "12V_EN" input
+		(pin "9V_EN" input
 			(at 114.3 77.47 0)
 			(effects
@@
 		(pin "LED_ACT" bidirectional
 			(at 114.3 86.36 0)
+			(effects
+				(font
+					(size 1.27 1.27)
+				)
+				(justify right)
+			)
+		)
+		(pin "~{POWER_SAVE}" input
+			(at 114.3 81.28 0)
 			(effects
 				(font
@@
 		)
 		(pin "RS485_TX" input
+			(at 114.3 111.76 0)
+			(effects
+				(font
+					(size 1.27 1.27)
+				)
+				(justify right)
+			)
+		)
+		(pin "RS485_RX" output
 			(at 114.3 109.22 0)
 			(effects
@@
 			)
 		)
-		(pin "RS485_RX" output
-			(at 114.3 106.68 0)
-			(effects
-				(font
-					(size 1.27 1.27)
-				)
-				(justify right)
-			)
-		)
-		(pin "RS485_DR" input
-			(at 114.3 99.06 0)
-			(effects
-				(font
+		(pin "~{RS485_RE}" input
+			(at 114.3 100.33 0)
+			(effects
+				(font
+					(size 1.27 1.27)
+				)
+				(justify right)
+			)
+		)
+		(pin "RS485_DE" input
+			(at 114.3 97.79 0)
+			(effects
+				(font
+					(size 1.27 1.27)
+				)
+				(justify right)
+			)
+		)
+		(pin "RS485_EN" input
+			(at 114.3 104.14 0)
+			(effects
+				(font
