File: Node_RS485/PSU.kicad_sch (KiCad schematic)
At the start: 51 parts, among them J3 CONN_PWRIN, Q3 APM4015P, Q4 SI2300, Q5 SI2301, U11 MT3608, U3 BQ24075RGT, U4 XL1509-5.0, U5 TPS63000, U7 DW01A, U8 FS8205A

Commit message: New version.
Parts:
- removed C19: 100nF, Footprints:C_0603, symbol Device:C_Small
- removed U7: DW01A, Footprints:SOT23-6, symbol Libraries:DW01A
- removed U8: FS8205A, Package_SO:TSSOP-8_4.4x3mm_P0.65mm, symbol Libraries:FS8205A
- added R33: 0R, Footprints:R_0603, symbol Device:R_Small
- R23: value 100R -> 4K7
- R24: value 1K -> 0R
- R36: value 10K -> 100K
- R37: value 10K -> 20K
- R39: value 51K -> 33K
Connections:
- net -BATT is gone; now on net GND: BT1.2 (-)
- net +BATT: no longer R23.1
- net GND: now also R33.2; no longer R24.1
- net at C11.2, R16.2, U5.6 (EN)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: no longer U5.7 (PS/SYNC)
- net at R23.2: now also R39.1
- net ~{POWER_SAVE}: now reaches R24.2
- net +12V renamed +9V
- net +9V: now also R23.1; no longer R39.1
- net 12V_EN renamed 9V_EN
- new net: R24.1, R33.1, U5.7 (PS/SYNC)
- no-connect marks 3 -> 1
Other:
- note added: "3V3 buck-boost converter"
- note added: "7-40V to 5V buck converter."
- note added: "BOOST 9V (RS485 Sensor)"
- note added: "Battery & Voltage sense"
- note added: "Power path manager"
- note removed: "8-40V TO 5V"
- note removed: "BATTERY PROTECTION - MONITOR"
- note removed: "BOOST 12V (RS485 Sensor)"
- note removed: "BUCK-BOOST TO 3V3"
- note removed: "POWER PATH MANAGEMENT IC"
- moved on the sheet: C11, C12, C15, C33, C34, C35, D7, L5, Q4, Q5, R16, R19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
