File: Node_RS485/RAK3172_LoRa.kicad_sch (KiCad schematic)
At the start: 14 parts, among them J1 RAK_DEBUG, Q1 SI2300, SW1 RAK-RESET, SW4 USER_BTN, U1 RAK3172

Commit message: New version.
Parts:
- R2: value 10K -> 100K
- R22, R3: value 10K -> 20K
- SW4: value USER_BTN -> MODE_SEL_BTN
Connections:
- net LED_ACT: now also U1.16 (SS/PA4); no longer U1.19 (PA8)
- net SENSOR_PWRON: now also U1.13 (MOSI/PA7); no longer U1.27 (PB12)
- net ~{POWER_SAVE}: now reaches U1.10 (SDA/PA11)
- net ~{RS485_RE}: now reaches U1.14 (MISO/PA6)
- net RS485_DE: now reaches U1.15 (SCK/PA5)
- net RS485_PWREN: now reaches U1.9 (SCL/PA12)
- net RS485_DR: no longer names the net of U1.6 (PA1)
- no-connect marks 12 -> 9
Other:
- moved on the sheet: C16, R22, SW4
Changed lines of the file:
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@@
 	(paper "A4")
 	(junction
-		(at 223.52 123.19)
+		(at 215.9 123.19)
 		(diameter 0)
 		(color 0 0 0 0)
@@
 	)
 	(junction
-		(at 223.52 110.49)
+		(at 215.9 110.49)
 		(diameter 0)
 		(color 0 0 0 0)
@@
 	)
 	(junction
-		(at 217.17 110.49)
+		(at 209.55 110.49)
 		(diameter 0)
 		(color 0 0 0 0)
@@
 	)
 	(no_connect
-		(at 198.12 90.17)
-	)
-	(no_connect
 		(at 198.12 102.87)
 	)
@@
 	)
 	(no_connect
-		(at 198.12 92.71)
+		(at 147.32 110.49)
 	)
 	(no_connect
-		(at 198.12 80.01)
+		(at 198.12 105.41)
 	)
 	(no_connect
@@
 	)
 	(no_connect
-		(at 198.12 77.47)
-	)
-	(no_connect
 		(at 147.32 87.63)
 	)
@@
 	)
 	(no_connect
-		(at 198.12 85.09)
-	)
-	(no_connect
-		(at 198.12 87.63)
-	)
-	(wire
-		(pts
-			(xy 223.52 124.46) (xy 223.52 123.19)
-		)
-		(stroke
-			(width 0)
-			(type default)
-		)
-	)
-	(wire
-		(pts
-			(xy 223.52 123.19) (xy 217.17 123.19)
+		(at 198.12 107.95)
+	)
+	(wire
+		(pts
+			(xy 215.9 124.46) (xy 215.9 123.19)
+		)
+		(stroke
+			(width 0)
+			(type default)
+		)
+	)
+	(wire
+		(pts
+			(xy 215.9 123.19) (xy 209.55 123.19)
 		)
 		(stroke
@@
 	(wire
 		(pts
-			(xy 223.52 111.76) (xy 223.52 110.49)
+			(xy 215.9 111.76) (xy 215.9 110.49)
 		)
 		(stroke
@@
 	(wire
 		(pts
-			(xy 223.52 109.22) (xy 223.52 110.49)
+			(xy 215.9 109.22) (xy 215.9 110.49)
 		)
 		(stroke
@@
 	(wire
 		(pts
-			(xy 217.17 119.38) (xy 217.17 123.19)
+			(xy 209.55 119.38) (xy 209.55 123.19)
 		)
 		(stroke
@@
 	(wire
 		(pts
-			(xy 198.12 110.49) (xy 217.17 110.49)
+			(xy 198.12 110.49) (xy 209.55 110.49)
 		)
 		(stroke
@@
 	(wire
 		(pts
-			(xy 217.17 110.49) (xy 217.17 114.3)
+			(xy 209.55 110.49) (xy 209.55 114.3)
 		)
 		(stroke
@@
 	(wire
 		(pts
-			(xy 223.52 121.92) (xy 223.52 123.19)
+			(xy 215.9 121.92) (xy 215.9 123.19)
 		)
 		(stroke
@@
 	(wire
 		(pts
-			(xy 223.52 110.49) (xy 217.17 110.49)
+			(xy 215.9 110.49) (xy 209.55 110.49)
 		)
 		(stroke
@@
 		)
 	)
-	(hierarchical_label "SENSOR_PWRON"
+	(hierarchical_label "RS485_DE"
 		(shape output)
-		(at 147.32 110.49 180)
+		(at 198.12 87.63 0)
 		(fields_autoplaced yes)
 		(effects
@@
 				(size 1.27 1.27)
 			)
-			(justify right)
+			(justify left)
+		)
+	)
+	(hierarchical_label "SENSOR_PWRON"
+		(shape output)
+		(at 198.12 92.71 0)
+		(fields_autoplaced yes)
+		(effects
+			(font
+				(size 1.27 1.27)
+			)
+			(justify left)
 		)
 	)
@@
 	(hierarchical_label "LED_ACT"
 		(shape bidirectional)
-		(at 198.12 107.95 0)
+		(at 198.12 85.09 0)
 		(fields_autoplaced yes)
 		(effects
@@
 		)
 	)
+	(hierarchical_label "RS485_PWREN"
+		(shape output)
+		(at 198.12 80.01 0)
+		(fields_autoplaced yes)
+		(effects
+			(font
+				(size 1.27 1.27)
+			)
+			(justify left)
+		)
+	)
+	(hierarchical_label "~{POWER_SAVE}"
+		(shape output)
+		(at 198.12 77.47 0)
+		(fields_autoplaced yes)
+		(effects
+			(font
+				(size 1.27 1.27)
+			)
+			(justify left)
+		)
+	)
 	(hierarchical_label "UART2_RX"
 		(shape input)
@@
 		)
 	)
-	(hierarchical_label "RS485_DR"
+	(hierarchical_label "~{RS485_RE}"
 		(shape output)
-		(at 198.12 105.41 0)
+		(at 198.12 90.17 0)
 		(fields_autoplaced yes)
 		(effects
@@
 			)
 		)
-		(property "Value" "10K"
+		(property "Value" "100K"
 			(at 90.932 83.82 0)
 			(effects
@@
 	(symbol
 		(lib_id "power:+3V3")
-		(at 223.52 104.14 0)
+		(at 215.9 104.14 0)
 		(mirror y)
 		(unit 1)
@@
 		(dnp no)
 		(property "Reference" "#PWR043"
-			(at 223.52 107.95 0)
+			(at 215.9 107.95 0)
 			(effects
 				(font
@@
 		)
 		(property "Value" "+3V3"
-			(at 223.52 100.584 0)
+			(at 215.9 100.584 0)
 			(effects
 				(font
@@
 		)
 		(property "Footprint" ""
-			(at 223.52 104.14 0)
+			(at 215.9 104.14 0)
 			(effects
 				(font
@@
 		)
 		(property "Datasheet" ""
-			(at 223.52 104.14 0)
+			(at 215.9 104.14 0)
 			(effects
 				(font
@@
 		)
 		(property "Description" "Power symbol creates a global label with name \"+3V3\""
-			(at 223.52 104.14 0)
+			(at 215.9 104.14 0)
 			(effects
 				(font
@@
 	(symbol
 		(lib_id "power:GND")
-		(at 223.52 124.46 0)
+		(at 215.9 124.46 0)
 		(mirror y)
 		(unit 1)
@@
 		(dnp no)
 		(property "Reference" "#PWR044"
-			(at 223.52 130.81 0)
+			(at 215.9 130.81 0)
 			(effects
 				(font
@@
 		)
 		(property "Value" "GND"
-			(at 223.52 128.27 0)
+			(at 215.9 128.27 0)
 			(effects
 				(font
@@
 		)
 		(property "Footprint" ""
-			(at 223.52 124.46 0)
+			(at 215.9 124.46 0)
 			(effects
 				(font
@@
 		)
 		(property "Datasheet" ""
-			(at 223.52 124.46 0)
+			(at 215.9 124.46 0)
 			(effects
 				(font
@@
 		)
 		(property "Description" "Power symbol creates a global label with name \"GND\" , ground"
-			(at 223.52 124.46 0)
+			(at 215.9 124.46 0)
 			(effects
 				(font
@@
 	(symbol
 		(lib_id "Device:C_Small")
-		(at 217.17 116.84 0)
+		(at 209.55 116.84 0)
 		(mirror y)
 		(unit 1)
@@
 		(dnp no)
 		(property "Reference" "C16"
-			(at 215.646 115.57 0)
+			(at 208.026 115.57 0)
 			(effects
 				(font
@@
 		)
 		(property "Value" "100nF"
-			(at 215.646 118.11 0)
+			(at 208.026 118.11 0)
 			(effects
 				(font
@@
 		)
 		(property "Footprint" "Footprints:C_0603"
-			(at 217.17 116.84 0)
+			(at 209.55 116.84 0)
 			(effects
 				(font
@@
 		)
 		(property "Datasheet" "~"
-			(at 217.17 116.84 0)
+			(at 209.55 116.84 0)
 			(effects
 				(font
@@
 		)
 		(property "Description" "Unpolarized capacitor, small symbol"
-			(at 217.17 116.84 0)
+			(at 209.55 116.84 0)
 			(effects
 				(font
@@
 	(symbol
 		(lib_id "Switch:SW_Push")
-		(at 223.52 116.84 270)
+		(at 215.9 116.84 270)
 		(mirror x)
 		(unit 1)
@@
 		(fields_autoplaced yes)
 		(property "Reference" "SW4"
-			(at 227.33 115.5699 90)
-			(effects
-				(font
-					(size 1.27 1.27)
-				)
-				(justify left)
-			)
-		)
-		(property "Value" "USER_BTN"
-			(at 227.33 118.1099 90)
+			(at 219.71 115.5699 90)
+			(effects
+				(font
+					(size 1.27 1.27)
+				)
+				(justify left)
+			)
+		)
+		(property "Value" "MODE_SEL_BTN"
+			(at 219.71 118.1099 90)
 			(effects
 				(font
@@
 		)
 		(property "Footprint" "Footprints:Switch_Tactile_6x6_Horizontal"
-			(at 228.6 116.84 0)
+			(at 220.98 116.84 0)
 			(effects
 				(font
@@
 		)
 		(property "Datasheet" "~"
-			(at 228.6 116.84 0)
+			(at 220.98 116.84 0)
 			(effects
 				(font
@@
 		)
 		(property "Description" "Push button switch, generic, two pins"
-			(at 223.52 116.84 0)
+			(at 215.9 116.84 0)
 			(effects
 				(font
@@
 			)
 		)
-		(property "Value" "10K"
+		(property "Value" "20K"
 			(at 113.792 69.85 0)
 			(effects
@@
 	(symbol
 		(lib_id "Device:R_Small")
-		(at 223.52 106.68 0)
+		(at 215.9 106.68 0)
 		(mirror y)
 		(unit 1)
@@
 		(dnp no)
 		(property "Reference" "R22"
-			(at 222.758 105.41 0)
-			(effects
-				(font
-					(size 1.27 1.27)
-				)
-				(justify left)
-			)
-		)
-		(property "Value" "10K"
-			(at 222.758 107.95 0)
+			(at 215.138 105.41 0)
+			(effects
+				(font
+					(size 1.27 1.27)
+				)
+				(justify left)
+			)
+		)
+		(property "Value" "20K"
+			(at 215.138 107.95 0)
 			(effects
 				(font
@@
 		)
 		(property "Footprint" "Footprints:R_0603"
-			(at 223.52 106.68 0)
+			(at 215.9 106.68 0)
 			(effects
 				(font
@@
 		)
 		(property "Datasheet" "~"
-			(at 223.52 106.68 0)
+			(at 215.9 106.68 0)
 			(effects
 				(font
@@
 		)
 		(property "Description" "Resistor, small symbol"
-			(at 223.52 106.68 0)
-			(effects
-				(font
+			(at 215.9 106.68 0)
+			(effects
+				(font
